Commit message: publishing topology

File: rotors_description/urdf/caric_firefly_base.xacro (robot description, xacro)
@@ -47,5 +47,5 @@
   <!-- </xacro:if> -->
   <!-- Mount a PPCom-sensor in the center of body. -->
-  <xacro:ppcom_plugin_macro
+  <!-- <xacro:ppcom_plugin_macro
       namespace="${namespace}"
       ppcom_suffix=""
@@ -58,4 +58,4 @@
     <inertia ixx="0.00001" ixy="0.0" ixz="0.0" iyy="0.00001" iyz="0.0" izz="0.00001" />
     <origin xyz="0.0 0.0 0.0" rpy="0 0 0" />
-  </xacro:ppcom_plugin_macro>
+  </xacro:ppcom_plugin_macro> -->
 </robot>

File: rotors_description/urdf/gcs_base.xacro (robot description, xacro)
@@ -36,5 +36,5 @@
     <link name="${robot_namespace}/base_link"></link>
     <joint name="${robot_namespace}/base_joint" type="fixed">
-      <origin xyz="0 0 0" rpy="0 0 0" />
+      <origin xyz="0 0 0" rpy="0 0 4.71238898038" />
       <parent link="${robot_namespace}/base_link" />
       <child link="${robot_namespace}/base_link_inertia" />

Commit message: some more features for ppcom

File: rotors_description/urdf/caric_firefly_base.xacro (robot description, xacro)
@@ -49,8 +49,8 @@
   <!-- <xacro:ppcom_plugin_macro
       namespace="${namespace}"
+      parent_link="${namespace}/base_link"
+      mass="0.015"
       ppcom_suffix=""
-      parent_link="${namespace}/base_link"
       ppcom_topic="ppcom"
-      mass_ppcom_sensor="0.015"
       ppcom_id="${ppcom_id}"
       ppcom_config="${ppcom_config}"
@@ -59,3 +59,8 @@
     <origin xyz="0.0 0.0 0.0" rpy="0 0 0" />
   </xacro:ppcom_plugin_macro> -->
+  <!-- <sensor name='my_contact' type='contact'>
+    <contact>
+      <collision>box_collision</collision>
+    </contact>
+  </sensor> -->
 </robot>

File: rotors_description/urdf/component_snippets.xacro (robot description, xacro)
@@ -824,6 +824,6 @@
     <!-- Macro to add a PPCom sensor. -->
     <xacro:macro name="ppcom_plugin_macro"
-        params="namespace ppcom_suffix parent_link ppcom_topic mass_ppcom_sensor
-                ppcom_id ppcom_config
+        params="namespace parent_link mass
+                ppcom_suffix ppcom_id ppcom_config ppcom_topic ppcom_hz
                 *inertia *origin">
         <!-- IMU link -->
@@ -831,5 +831,5 @@
             <inertial>
                 <xacro:insert_block name="inertia" />
-                <mass value="${mass_ppcom_sensor}" />  <!-- [kg] -->
+                <mass value="${mass}" />  <!-- [kg] -->
                 <origin xyz="0 0 0" rpy="0 0 0" />
             </inertial>
@@ -856,4 +856,6 @@
                 <!-- (string): Path to the network configuration of PPCom-->
                 <ppcomConfig>${ppcom_config}</ppcomConfig>
+                <!-- (double): Update period of the ppcom -->
+                <ppcomHz>${ppcom_hz}</ppcomHz>
             </plugin>
         </gazebo>

File: rotors_description/urdf/gcs.xacro (robot description, xacro)
@@ -21,4 +21,5 @@
   <xacro:property name="ppcom_id"      value="$(arg ppcom_id)" />
   <xacro:property name="ppcom_config"  value="$(arg ppcom_config)" />
+  <xacro:property name="ppcom_hz"      value="$(arg ppcom_hz)" />
   <xacro:property name="use_mesh_file" value="true" />
   <xacro:property name="mesh_file"     value="package://rotors_description/meshes/gcs/gcs.dae" />
@@ -58,10 +59,11 @@
   <xacro:ppcom_plugin_macro
       namespace="${namespace}"
+      parent_link="${namespace}/base_link"
+      mass="0.015"
       ppcom_suffix=""
-      parent_link="${namespace}/base_link"
       ppcom_topic="ppcom"
-      mass_ppcom_sensor="0.015"
       ppcom_id="${ppcom_id}"
       ppcom_config="${ppcom_config}"
+      ppcom_hz="${ppcom_hz}"
   >
     <inertia ixx="0.00001" ixy="0.0" ixz="0.0" iyy="0.00001" iyz="0.0" izz="0.00001" />

File: rotors_description/urdf/gcs_base.xacro (robot description, xacro)
@@ -60,5 +60,5 @@
         <origin xyz="0 0 0" rpy="0 0 0" />
         <geometry>
-          <box size="${body_width} ${body_width} ${body_height}" /> <!-- [m] [m] [m] -->
+          <box size="${body_width} ${body_width} ${body_height}" />
         </geometry>
       </collision>

Commit message: fixed the lidar plugin

File: rotors_description/urdf/caric_firefly_base.xacro (robot description, xacro)
@@ -64,3 +64,13 @@
     </contact>
   </sensor> -->
+  <!-- Mount a lidar sensor -->
+  <xacro:lidars_plugin_macro
+      namespace="${namespace}"
+      parent_link="${namespace}/base_link"
+      mass="0.01"
+      lidar_suffix=""
+  >
+    <inertia ixx="0.00001" ixy="0.0" ixz="0.0" iyy="0.00001" iyz="0.0" izz="0.00001" />
+    <origin xyz="0.0 0.0 0.0" rpy="0 0 0" />
+  </xacro:lidars_plugin_macro>
 </robot>

File: rotors_description/urdf/component_snippets.xacro (robot description, xacro)
@@ -861,4 +861,60 @@
         </gazebo>
     </xacro:macro>
+    <!-- Macro to add a lidar -->
+    <xacro:macro name="lidars_plugin_macro"
+        params="namespace parent_link mass lidar_suffix
+                *inertia *origin">
+        <!-- IMU link -->
+        <link name="${namespace}/lidar${lidar_suffix}_link">
+            <inertial>
+                <xacro:insert_block name="inertia" />
+                <mass value="${mass}" />  <!-- [kg] -->
+                <origin xyz="0 0 0" rpy="0 0 0" />
+            </inertial>
+        </link>
+        <!-- IMU joint -->
+        <joint name="${namespace}/lidar${lidar_suffix}_joint" type="revolute">
+            <xacro:insert_block name="origin" />
+            <parent link="${parent_link}" />
+            <child link="${namespace}/lidar${lidar_suffix}_link" />
+            <limit upper="0" lower="0" effort="0" velocity="0" />
+        </joint>
+        <gazebo reference="${namespace}/lidar${lidar_suffix}_link">
+            <sensor name="laser" type="ray">
+                <pose>0 0 0.3 0 0 0</pose>
+                <ray>
+                    <scan>
+                        <horizontal>
+                            <samples>1024</samples>
+                            <resolution>1</resolution>
+                            <min_angle>0</min_angle>
+                            <max_angle>6.29</max_angle>
+                        </horizontal>
+                        <vertical>
+                            <samples>16</samples>
+                            <resolution>1</resolution>
+                            <min_angle>-0.39269908169</min_angle>
+                            <max_angle>0.39269908169</max_angle>
+                        </vertical>
+                    </scan>
+                    <range>
+                        <min>0.06</min>
+                        <max>25</max>
+                        <resolution>0.01</resolution>
+                    </range>
+                    <noise>
+                        <type>gaussian</type>
+                        <mean>0.0</mean>
+                        <stddev>0.01</stddev>
+                    </noise>
+                </ray>
+                <plugin name="LaserPlugin" filename="librotors_gazebo_lidar_plugin.so"/>
+                <robotNamespace>${namespace}</robotNamespace>
+                <always_on>1</always_on>
+                <update_rate>1</update_rate>
+                <visualize>false</visualize>
+            </sensor>
+        </gazebo>
+    </xacro:macro>
     <xacro:macro name="ground_truth_imu_and_odometry" params="namespace parent_link">
         <!-- Mount an IMU providing ground truth. -->

Commit message: tidied up

File: rotors_description/urdf/caric_firefly_base.xacro (robot description, xacro)
@@ -65,5 +65,5 @@
   </sensor> -->
   <!-- Mount a lidar sensor -->
-  <xacro:lidars_plugin_macro
+  <!-- <xacro:lidars_plugin_macro
       namespace="${namespace}"
       parent_link="${namespace}/base_link"
@@ -73,4 +73,8 @@
     <inertia ixx="0.00001" ixy="0.0" ixz="0.0" iyy="0.00001" iyz="0.0" izz="0.00001" />
     <origin xyz="0.0 0.0 0.0" rpy="0 0 0" />
-  </xacro:lidars_plugin_macro>
+  </xacro:lidars_plugin_macro> -->
+  <xacro:include filename="$(find velodyne_description)/urdf/VLP-16.urdf.xacro"/>
+  <xacro:VLP-16 parent="${namespace}/base_link" name="velodyne" topic="/${namespace}/velodyne_points" hz="10" samples="440" gpu="true">
+    <origin xyz="0 0 0.2" rpy="0 0 0" />
+  </xacro:VLP-16>
 </robot>

File: rotors_description/urdf/component_snippets.xacro (robot description, xacro)
@@ -862,4 +862,6 @@
     </xacro:macro>
     <!-- Macro to add a lidar -->
+    <!-- horz_sample horz_res horz_anglemin horz_anglemax
+    vert_sample vert_res vert_anglemin vert_anglemax -->
     <xacro:macro name="lidars_plugin_macro"
         params="namespace parent_link mass lidar_suffix
@@ -886,5 +888,5 @@
                     <scan>
                         <horizontal>
-                            <samples>1024</samples>
+                            <samples>2</samples>
                             <resolution>1</resolution>
                             <min_angle>0</min_angle>
@@ -892,5 +894,5 @@
                         </horizontal>
                         <vertical>
-                            <samples>16</samples>
+                            <samples>2</samples>
                             <resolution>1</resolution>
                             <min_angle>-0.39269908169</min_angle>
@@ -900,5 +902,5 @@
                     <range>
                         <min>0.06</min>
-                        <max>25</max>
+                        <max>50</max>
                         <resolution>0.01</resolution>
                     </range>
@@ -912,6 +914,6 @@
                 <robotNamespace>${namespace}</robotNamespace>
                 <always_on>1</always_on>
-                <update_rate>1</update_rate>
-                <visualize>false</visualize>
+                <update_rate>0.25</update_rate>
+                <visualize>true</visualize>
             </sensor>
         </gazebo>

File: rotors_description/urdf/gcs.xacro (robot description, xacro)
@@ -74,5 +74,5 @@
     <origin xyz="0.0 0.0 0.0" rpy="0 0 0" />
   </xacro:ppcom_plugin_macro>
-  <xacro:caric_plugin_macro
+  <!-- <xacro:caric_plugin_macro
       namespace="${namespace}"
       parent_link="${namespace}/base_link"
@@ -88,4 +88,4 @@
     <inertia ixx="0.00001" ixy="0.0" ixz="0.0" iyy="0.00001" iyz="0.0" izz="0.00001" />
     <origin xyz="0.0 0.0 0.0" rpy="0 0 0" />
-  </xacro:caric_plugin_macro>
+  </xacro:caric_plugin_macro> -->
 </robot>

Commit message: added servo and attached lidar to servo

File: rotors_description/urdf/caric_firefly_base.xacro (robot description, xacro)
@@ -74,7 +74,22 @@
     <origin xyz="0.0 0.0 0.0" rpy="0 0 0" />
   </xacro:lidars_plugin_macro> -->
+  <xacro:include filename="$(find rotors_description)/urdf/servo.xacro" />
+  <xacro:servo
+    namespace="${namespace}"
+    suffix=""
+    parent="${namespace}/base_link"
+    mass_servo="0.05"
+    rotating_period="8.0"
+  >
+    <origin xyz="0.2 0 0.2" rpy="0 0 0" />
+    <inertia ixx="0.00001" ixy="0.0" ixz="0.0" iyy="0.00001" iyz="0.0" izz="0.00001" />
+    <!-- <xacro:insert_block name="rotor_inertia" /> -->
+  </xacro:servo>
   <xacro:include filename="$(find velodyne_description)/urdf/VLP-16.urdf.xacro"/>
-  <xacro:VLP-16 parent="${namespace}/base_link" name="velodyne" topic="/${namespace}/velodyne_points" hz="10" samples="440" gpu="true">
-    <origin xyz="0 0 0.2" rpy="0 0 0" />
+  <xacro:VLP-16 parent="${namespace}/servo"
+                name="velodyne" topic="/${namespace}/velodyne_points"
+                max_range="65.0" noise="0.0" hz="10" samples="440" gpu="true">
+    <origin xyz="0.0 0.0 -0.03585" rpy="0 0 0" />
+    <!-- <origin xyz="0.0 0.0 0.2" rpy="1.57079632679 0 0" /> -->
   </xacro:VLP-16>
 </robot>

File: rotors_description/urdf/component_snippets.xacro (robot description, xacro)
@@ -984,5 +984,5 @@
         <xacro:odometry_plugin_macro
             namespace="${namespace}"
-            odometry_sensor_suffix="gt"
+            odometry_sensor_suffix=""
             parent_link="${parent_link}"
             pose_topic="ground_truth/pose"
