Commit message: successful ray tracing

File: rotors_description/urdf/component_snippets.xacro (robot description, xacro)
@@ -17,236 +17,238 @@
 -->
 <robot xmlns:xacro="http://ros.org/wiki/xacro">
-  <!-- Macro to add logging to a bag file. -->
-  <xacro:macro name="bag_plugin_macro"
-    params="namespace bag_file rotor_velocity_slowdown_sim wait_to_record_bag">
-    <gazebo>
-      <plugin filename="librotors_gazebo_bag_plugin.so" name="rosbag">
-        <robotNamespace>${namespace}</robotNamespace>
-        <bagFileName>${bag_file}</bagFileName>
-        <linkName>${namespace}/base_link</linkName>
-        <frameId>${namespace}/base_link</frameId>
-        <rotorVelocitySlowdownSim>${rotor_velocity_slowdown_sim}</rotorVelocitySlowdownSim>
-	<waitToRecordBag>${wait_to_record_bag}</waitToRecordBag>
-      </plugin>
-    </gazebo>
-  </xacro:macro>
-  <!-- Macro to add a camera. -->
-  <xacro:macro name="camera_macro"
-    params="namespace parent_link camera_suffix frame_rate
+    <!-- Macro to add logging to a bag file. -->
+    <xacro:macro name="bag_plugin_macro"
+        params="namespace bag_file rotor_velocity_slowdown_sim wait_to_record_bag">
+        <gazebo>
+            <plugin filename="librotors_gazebo_bag_plugin.so" name="rosbag">
+                <robotNamespace>${namespace}</robotNamespace>
+                <bagFileName>${bag_file}</bagFileName>
+                <linkName>${namespace}/base_link</linkName>
+                <frameId>${namespace}/base_link</frameId>
+                <rotorVelocitySlowdownSim>${rotor_velocity_slowdown_sim}</rotorVelocitySlowdownSim>
+                <waitToRecordBag>${wait_to_record_bag}</waitToRecordBag>
+            </plugin>
+        </gazebo>
+    </xacro:macro>
+    <!-- Macro to add a camera. -->
+    <xacro:macro name="camera_macro"
+        params="namespace parent_link camera_suffix frame_rate
       horizontal_fov image_width image_height image_format min_distance
       max_distance noise_mean noise_stddev enable_visual *geometry *origin">
-    <link name="${namespace}/camera_${camera_suffix}_link">
-      <collision>
-        <origin xyz="0 0 0" rpy="0 0 0" />
-        <geometry>
-          <xacro:insert_block name="geometry" />
-        </geometry>
-      </collision>
-      <xacro:if value="${enable_visual}">
-        <visual>
-          <origin xyz="0 0 0" rpy="0 ${pi/2} 0" />
-          <geometry>
-            <xacro:insert_block name="geometry" />
-          </geometry>
-          <material name="red" />
-        </visual>
-      </xacro:if>
-      <inertial>
-        <mass value="1e-5" />
-        <origin xyz="0 0 0" rpy="0 0 0" />
-        <inertia ixx="1e-6" ixy="0" ixz="0" iyy="1e-6" iyz="0" izz="1e-6" />
-      </inertial>
-    </link>
-    <joint name="${namespace}/camera_${camera_suffix}_joint" type="fixed">
-      <xacro:insert_block name="origin" />
-      <parent link="${parent_link}" />
-      <child link="${namespace}/camera_${camera_suffix}_link" />
-    </joint>
-    <link name="${namespace}/camera_${camera_suffix}_optical_link" />
-    <joint name="${namespace}/camera_${camera_suffix}_optical_joint" type="fixed" >
-      <origin xyz="0 0 0" rpy="${-pi/2} 0 ${-pi/2}" />
-      <parent link="${namespace}/camera_${camera_suffix}_link" />
-      <child link="${namespace}/camera_${camera_suffix}_optical_link" />
-    </joint>
-    <gazebo reference="${namespace}/camera_${camera_suffix}_link">
-      <sensor type="camera" name="${namespace}_camera_${camera_suffix}">
-        <update_rate>${frame_rate}</update_rate>
-        <camera name="head">
-          <horizontal_fov>${horizontal_fov}</horizontal_fov>
-          <image>
-            <width>${image_width}</width>
-            <height>${image_height}</height>
-            <format>${image_format}</format>
-          </image>
-          <clip>
-            <near>${min_distance}</near>
-            <far>${max_distance}</far>
-          </clip>
-          <noise>
-            <type>gaussian</type>
-            <!-- Noise is sampled independently per pixel on each frame.
+        <link name="${namespace}/camera_${camera_suffix}_link">
+            <collision>
+                <origin xyz="0 0 0" rpy="0 0 0" />
+                <geometry>
+                    <xacro:insert_block name="geometry" />
+                </geometry>
+            </collision>
+            <xacro:if value="${enable_visual}">
+                <visual>
+                    <origin xyz="0 0 0" rpy="0 ${pi/2} 0" />
+                    <geometry>
+                        <xacro:insert_block name="geometry" />
+                    </geometry>
+                    <material name="red" />
+                </visual>
+            </xacro:if>
+            <inertial>
+                <mass value="1e-5" />
+                <origin xyz="0 0 0" rpy="0 0 0" />
+                <inertia ixx="1e-6" ixy="0" ixz="0" iyy="1e-6" iyz="0" izz="1e-6" />
+            </inertial>
+        </link>
+        <joint name="${namespace}/camera_${camera_suffix}_joint" type="fixed">
+            <xacro:insert_block name="origin" />
+            <parent link="${parent_link}" />
+            <child link="${namespace}/camera_${camera_suffix}_link" />
+        </joint>
+        <link name="${namespace}/camera_${camera_suffix}_optical_link" />
+        <joint name="${namespace}/camera_${camera_suffix}_optical_joint" type="fixed">
+            <origin xyz="0 0 0" rpy="${-pi/2} 0 ${-pi/2}" />
+            <parent link="${namespace}/camera_${camera_suffix}_link" />
+            <child link="${namespace}/camera_${camera_suffix}_optical_link" />
+        </joint>
+        <gazebo reference="${namespace}/camera_${camera_suffix}_link">
+            <sensor type="camera" name="${namespace}_camera_${camera_suffix}">
+                <update_rate>${frame_rate}</update_rate>
+                <camera name="head">
+                    <horizontal_fov>${horizontal_fov}</horizontal_fov>
+                    <image>
+                        <width>${image_width}</width>
+                        <height>${image_height}</height>
+                        <format>${image_format}</format>
+                    </image>
+                    <clip>
+                        <near>${min_distance}</near>
+                        <far>${max_distance}</far>
+                    </clip>
+                    <noise>
+                        <type>gaussian</type>
+                        <!-- Noise is sampled independently per pixel on each frame.
                  That pixel's noise value is added to each of its color
                  channels, which at that point lie in the range [0,1]. -->
-            <mean>${noise_mean}</mean>
-            <stddev>${noise_stddev}</stddev>
-          </noise>
-        </camera>
-        <plugin name="${namespace}_camera_${camera_suffix}_controller" filename="libgazebo_ros_camera.so">
-          <robotNamespace>${namespace}</robotNamespace>
-          <alwaysOn>true</alwaysOn>
-          <updateRate>${frame_rate}</updateRate>
-          <cameraName>camera_${camera_suffix}</cameraName>
-          <imageTopicName>image_raw</imageTopicName>
-          <cameraInfoTopicName>camera_info</cameraInfoTopicName>
-          <frameName>camera_${camera_suffix}_link</frameName>
-          <hackBaseline>0.0</hackBaseline>
-          <distortionK1>0.0</distortionK1>
-          <distortionK2>0.0</distortionK2>
-          <distortionK3>0.0</distortionK3>
-          <distortionT1>0.0</distortionT1>
-          <distortionT2>0.0</distortionT2>
-        </plugin>
-      </sensor>
-    </gazebo>
-  </xacro:macro>
-  <!-- Camera joint macro - just the joints, links, and collisions for a single
+                        <mean>${noise_mean}</mean>
+                        <stddev>${noise_stddev}</stddev>
+                    </noise>
+                </camera>
+                <plugin name="${namespace}_camera_${camera_suffix}_controller"
+                    filename="libgazebo_ros_camera.so">
+                    <robotNamespace>${namespace}</robotNamespace>
+                    <alwaysOn>true</alwaysOn>
+                    <updateRate>${frame_rate}</updateRate>
+                    <cameraName>camera_${camera_suffix}</cameraName>
+                    <imageTopicName>image_raw</imageTopicName>
+                    <cameraInfoTopicName>camera_info</cameraInfoTopicName>
+                    <frameName>camera_${camera_suffix}_link</frameName>
+                    <hackBaseline>0.0</hackBaseline>
+                    <distortionK1>0.0</distortionK1>
+                    <distortionK2>0.0</distortionK2>
+                    <distortionK3>0.0</distortionK3>
+                    <distortionT1>0.0</distortionT1>
+                    <distortionT2>0.0</distortionT2>
+                </plugin>
+            </sensor>
+        </gazebo>
+    </xacro:macro>
+    <!-- Camera joint macro - just the joints, links, and collisions for a single
        camera. -->
-  <xacro:macro name="camera_joint_macro"
-    params="namespace parent_link camera_suffix enable_visual *origin *geometry" >
-    <link name="${namespace}/camera_${camera_suffix}_link">
-      <collision>
-        <origin xyz="0 0 0" rpy="0 0 0" />
-        <geometry>
-          <xacro:insert_block name="geometry" />
-        </geometry>
-      </collision>
-      <xacro:if value="${enable_visual}">
-        <visual>
-          <origin xyz="0 0 0" rpy="0 0 0" />
-          <geometry>
-            <xacro:insert_block name="geometry" />
-          </geometry>
-          <material name="red" />
-        </visual>
-      </xacro:if>
-      <inertial>
-        <mass value="1e-5" />
-        <origin xyz="0 0 0" rpy="0 0 0" />
-        <inertia ixx="1e-6" ixy="0" ixz="0" iyy="1e-6" iyz="0" izz="1e-6" />
-      </inertial>
-    </link>
-    <joint name="${namespace}/camera_${camera_suffix}_joint" type="fixed">
-      <xacro:insert_block name="origin" />
-      <parent link="${parent_link}" />
-      <child link="${namespace}/camera_${camera_suffix}_link" />
-    </joint>
-  </xacro:macro>
-  <!-- Camera sensor macro - just image parameters. -->
-  <xacro:macro name="camera_sensor_macro"
-    params="camera_suffix horizontal_fov image_width image_height
+    <xacro:macro name="camera_joint_macro"
+        params="namespace parent_link camera_suffix enable_visual *origin *geometry">
+        <link name="${namespace}/camera_${camera_suffix}_link">
+            <collision>
+                <origin xyz="0 0 0" rpy="0 0 0" />
+                <geometry>
+                    <xacro:insert_block name="geometry" />
+                </geometry>
+            </collision>
+            <xacro:if value="${enable_visual}">
+                <visual>
+                    <origin xyz="0 0 0" rpy="0 0 0" />
+                    <geometry>
+                        <xacro:insert_block name="geometry" />
+                    </geometry>
+                    <material name="red" />
+                </visual>
+            </xacro:if>
+            <inertial>
+                <mass value="1e-5" />
+                <origin xyz="0 0 0" rpy="0 0 0" />
+                <inertia ixx="1e-6" ixy="0" ixz="0" iyy="1e-6" iyz="0" izz="1e-6" />
+            </inertial>
+        </link>
+        <joint name="${namespace}/camera_${camera_suffix}_joint" type="fixed">
+            <xacro:insert_block name="origin" />
+            <parent link="${parent_link}" />
+            <child link="${namespace}/camera_${camera_suffix}_link" />
+        </joint>
+    </xacro:macro>
+    <!-- Camera sensor macro - just image parameters. -->
+    <xacro:macro name="camera_sensor_macro"
+        params="camera_suffix horizontal_fov image_width image_height
       image_format min_distance max_distance noise_mean noise_stddev
-      baseline" >
-    <camera name="${camera_suffix}">
-      <pose>0 ${-baseline} 0 0 0 0</pose>
-      <horizontal_fov>${horizontal_fov}</horizontal_fov>
-      <image>
-        <width>${image_width}</width>
-        <height>${image_height}</height>
-        <format>${image_format}</format>
-      </image>
-      <clip>
-        <near>${min_distance}</near>
-        <far>${max_distance}</far>
-      </clip>
-      <noise>
-        <type>gaussian</type>
-        <!-- Noise is sampled independently per pixel on each frame.
+      baseline">
+        <camera name="${camera_suffix}">
+            <pose>0 ${-baseline} 0 0 0 0</pose>
+            <horizontal_fov>${horizontal_fov}</horizontal_fov>
+            <image>
+                <width>${image_width}</width>
+                <height>${image_height}</height>
+                <format>${image_format}</format>
+            </image>
+            <clip>
+                <near>${min_distance}</near>
+                <far>${max_distance}</far>
+            </clip>
+            <noise>
+                <type>gaussian</type>
+                <!-- Noise is sampled independently per pixel on each frame.
              That pixel's noise value is added to each of its color
              channels, which at that point lie in the range [0,1]. -->
-        <mean>${noise_mean}</mean>
-        <stddev>${noise_stddev}</stddev>
-      </noise>
-    </camera>
-  </xacro:macro>
-  <!-- Macro to add a multicamera (stereo pair). -->
-  <xacro:macro name="stereo_camera_macro"
-    params="namespace camera_name parent_link frame_rate
+                <mean>${noise_mean}</mean>
+                <stddev>${noise_stddev}</stddev>
+            </noise>
+        </camera>
+    </xacro:macro>
+    <!-- Macro to add a multicamera (stereo pair). -->
+    <xacro:macro name="stereo_camera_macro"
+        params="namespace camera_name parent_link frame_rate
       horizontal_fov image_width image_height image_format min_distance
       max_distance noise_mean noise_stddev enable_visual origin_offset_x
       baseline_y origin_offset_z *geometry">
-    <!-- These are parameters for the left camera link and then the right
+        <!-- These are parameters for the left camera link and then the right
         as well. -->
-    <xacro:camera_joint_macro namespace="${namespace}"
-      parent_link="${parent_link}"
-      camera_suffix="left" enable_visual="${enable_visual}">
-      <origin xyz="${origin_offset_x} ${baseline_y/2} ${origin_offset_z}" rpy="0 0 0" />
-      <xacro:insert_block name="geometry" />
-    </xacro:camera_joint_macro>
-    <xacro:camera_joint_macro namespace="${namespace}"
-      parent_link="${parent_link}"
-      camera_suffix="right" enable_visual="${enable_visual}">
-      <origin xyz="${origin_offset_x} ${-baseline_y/2} ${origin_offset_z}" rpy="0 0 0" />
-      <xacro:insert_block name="geometry" />
-    </xacro:camera_joint_macro>
-    <link name="${namespace}/camera_left_optical_link" />
-    <joint name="${namespace}/camera_left_optical_joint" type="fixed" >
-      <origin xyz="0 0 0" rpy="${-pi/2} 0 ${-pi/2}" />
-      <parent link="${namespace}/camera_left_link" />
-      <child link="${namespace}/camera_left_optical_link" />
-    </joint>
-    <!-- Both cameras in the pair are anchored off the left camera frame. -->
-    <gazebo reference="${namespace}/camera_left_link">
-      <sensor type="multicamera" name="${namespace}_stereo_camera">
-        <update_rate>${frame_rate}</update_rate>
-        <!-- Here we set up the individual cameras of the stereo head. -->
-        <xacro:camera_sensor_macro camera_suffix="left"
-            horizontal_fov="${horizontal_fov}" image_width="${image_width}"
-            image_height="${image_height}" image_format="${image_format}"
-            min_distance="${min_distance}" max_distance="${max_distance}"
-            noise_mean="${noise_mean}" noise_stddev="${noise_stddev}"
-            baseline="0">
-        </xacro:camera_sensor_macro>
-        <xacro:camera_sensor_macro camera_suffix="right"
-            horizontal_fov="${horizontal_fov}" image_width="${image_width}"
-            image_height="${image_height}" image_format="${image_format}"
-            min_distance="${min_distance}" max_distance="${max_distance}"
-            noise_mean="${noise_mean}" noise_stddev="${noise_stddev}"
-            baseline="${baseline_y}">
-        </xacro:camera_sensor_macro>
-        <!-- Stereo controller, setting the transforms between the two cameras. -->
-        <plugin name="${namespace}_stereo_camera_controller" filename="libgazebo_ros_multicamera.so">
-          <alwaysOn>true</alwaysOn>
-          <updateRate>0.0</updateRate>
-          <cameraName>${camera_name}</cameraName>
-          <imageTopicName>image_raw</imageTopicName>
-          <cameraInfoTopicName>camera_info</cameraInfoTopicName>
-          <frameName>${camera_name}/camera_left_link</frameName>
-          <hackBaseline>${baseline_y}</hackBaseline>
-          <distortionK1>0.0</distortionK1>
-          <distortionK2>0.0</distortionK2>
-          <distortionK3>0.0</distortionK3>
-          <distortionT1>0.0</distortionT1>
-          <distortionT2>0.0</distortionT2>
-        </plugin>
-      </sensor>
-    </gazebo>
-  </xacro:macro>
-  <!-- Macro to add the controller interface. -->
-  <xacro:macro name="controller_plugin_macro" params="namespace imu_sub_topic">
-    <gazebo>
-      <plugin name="controller_interface" filename="librotors_gazebo_controller_interface.so">
-        <robotNamespace>${namespace}</robotNamespace>
-        <commandAttitudeThrustSubTopic>command/attitude</commandAttitudeThrustSubTopic>
-        <commandRateThrustSubTopic>command/rate</commandRateThrustSubTopic>
-        <commandMotorSpeedSubTopic>command/motor_speed</commandMotorSpeedSubTopic>
-        <imuSubTopic>${imu_sub_topic}</imuSubTopic>
-        <motorSpeedCommandPubTopic>gazebo/command/motor_speed</motorSpeedCommandPubTopic>
-      </plugin>
-    </gazebo>
-  </xacro:macro>
-  <!-- =============================================================== -->
-  <!-- ==================== ROS INTERFACE MACRO ====================== -->
-  <!-- =============================================================== -->
-  <!-- <xacro:macro
+        <xacro:camera_joint_macro namespace="${namespace}"
+            parent_link="${parent_link}"
+            camera_suffix="left" enable_visual="${enable_visual}">
+            <origin xyz="${origin_offset_x} ${baseline_y/2} ${origin_offset_z}" rpy="0 0 0" />
+            <xacro:insert_block name="geometry" />
+        </xacro:camera_joint_macro>
+        <xacro:camera_joint_macro namespace="${namespace}"
+            parent_link="${parent_link}"
+            camera_suffix="right" enable_visual="${enable_visual}">
+            <origin xyz="${origin_offset_x} ${-baseline_y/2} ${origin_offset_z}" rpy="0 0 0" />
+            <xacro:insert_block name="geometry" />
+        </xacro:camera_joint_macro>
+        <link name="${namespace}/camera_left_optical_link" />
+        <joint name="${namespace}/camera_left_optical_joint" type="fixed">
+            <origin xyz="0 0 0" rpy="${-pi/2} 0 ${-pi/2}" />
+            <parent link="${namespace}/camera_left_link" />
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
Commit message: add caric camera evaluation plugin

File: rotors_description/urdf/component_snippets.xacro (robot description, xacro)
@@ -861,4 +861,46 @@
         </gazebo>
     </xacro:macro>
+    <!-- Macro to add a caric sensor. -->
+    <xacro:macro name="caric_plugin_macro"
+        params="namespace parent_link mass
+                ppcom_config interest_config ppcom_topic ppcom_hz
+                cam_x cam_y cam_z
+                *inertia *origin">
+        <!-- IMU link -->
+        <link name="${namespace}/caric_link">
+            <inertial>
+                <xacro:insert_block name="inertia" />
+                <mass value="${mass}" />  <!-- [kg] -->
+                <origin xyz="0 0 0" rpy="0 0 0" />
+            </inertial>
+        </link>
+        <!-- IMU joint -->
+        <joint name="${namespace}/caric_joint" type="revolute">
+            <xacro:insert_block name="origin" />
+            <parent link="${parent_link}" />
+            <child link="${namespace}/caric_link" />
+            <limit upper="0" lower="0" effort="0" velocity="0" />
+        </joint>
+        <gazebo>
+            <plugin filename="librotors_gazebo_caric_plugin.so" name="rotors_gazebo_caric_plugin">
+                <!-- A good description of the IMU parameters can be found in the kalibr
+                documentation: https://github.com/ethz-asl/kalibr/wiki/IMU-Noise-Model-and-Intrinsics -->
+                <!-- (string, required): ros namespace in which the messages are published -->
+                <robotNamespace>${namespace}</robotNamespace>
+                <!-- (string, required): name of the body which holds the IMU sensor -->
+                <linkName>${namespace}/caric_link</linkName>
+                <!-- (string): name of the sensor output topic and prefix of service names (defaults to ppcom) -->
+                <ppcomTopic>${ppcom_topic}</ppcomTopic>
+                <!-- (string): Path to the network configuration of PPCom-->
+                <ppcomConfig>${ppcom_config}</ppcomConfig>
+                <!-- (double): Update period of the ppcom -->
+                <ppcomHz>${ppcom_hz}</ppcomHz>
+                <interestPcd>${interest_config}</interestPcd>
+                <cam_x>${cam_x}</cam_x>
+                <cam_y>${cam_y}</cam_y>
+                <cam_z>${cam_z}</cam_z>
+            </plugin>
+        </gazebo>
+    </xacro:macro>
     <xacro:macro name="ground_truth_imu_and_odometry" params="namespace parent_link">
         <!-- Mount an IMU providing ground truth. -->

File: rotors_description/urdf/gcs.xacro (robot description, xacro)
@@ -22,4 +22,8 @@
   <xacro:property name="ppcom_config"  value="$(arg ppcom_config)" />
   <xacro:property name="ppcom_hz"      value="$(arg ppcom_hz)" />
+  <xacro:property name="interest_config"  value="$(arg interest_config)" />
+  <xacro:property name="cam_x"      value="$(arg cam_x)" />
+  <xacro:property name="cam_y"      value="$(arg cam_y)" />
+  <xacro:property name="cam_z"      value="$(arg cam_z)" />
   <xacro:property name="use_mesh_file" value="true" />
   <xacro:property name="mesh_file"     value="package://rotors_description/meshes/gcs/gcs.dae" />
@@ -70,3 +74,18 @@
     <origin xyz="0.0 0.0 0.0" rpy="0 0 0" />
   </xacro:ppcom_plugin_macro>
+  <xacro:caric_plugin_macro
+      namespace="${namespace}"
+      parent_link="${namespace}/base_link"
+      mass="0.015"
+      ppcom_config="${ppcom_config}"
+      interest_config="${interest_config}"
+      ppcom_topic="ppcom"
+      ppcom_hz="${ppcom_hz}"
+      cam_x="${cam_x}"
+      cam_y="${cam_y}"
+      cam_z="${cam_z}"
+  >
+    <inertia ixx="0.00001" ixy="0.0" ixz="0.0" iyy="0.00001" iyz="0.0" izz="0.00001" />
+    <origin xyz="0.0 0.0 0.0" rpy="0 0 0" />
+  </xacro:caric_plugin_macro>
 </robot>
