Commit message: revised the interest point name

File: rotors_description/urdf/component_snippets.xacro (robot description, xacro)
@@ -825,5 +825,5 @@
     <xacro:macro name="ppcom_plugin_macro"
         params="namespace parent_link mass
-                ppcom_suffix ppcom_id ppcom_config ppcom_topic ppcom_hz interest_config
+                ppcom_suffix ppcom_id ppcom_config ppcom_topic ppcom_hz interest_points
                 *inertia *origin">
         <!-- IMU link -->
@@ -858,5 +858,5 @@
                 <!-- (double): Update period of the ppcom -->
                 <ppcomHz>${ppcom_hz}</ppcomHz>
-                <interestPcd>${interest_config}</interestPcd>
+                <interestPcd>${interest_points}</interestPcd>
             </plugin>
         </gazebo>
@@ -923,5 +923,5 @@
     <xacro:macro name="caric_plugin_macro"
         params="namespace parent_link mass
-                ppcom_config interest_config ppcom_topic ppcom_hz
+                ppcom_config interest_points ppcom_topic ppcom_hz
                 cam_x cam_y cam_z
                 *inertia *origin">
@@ -955,5 +955,5 @@
                 <!-- (double): Update period of the ppcom -->
                 <ppcomHz>${ppcom_hz}</ppcomHz>
-                <interestPcd>${interest_config}</interestPcd>
+                <interestPcd>${interest_points}</interestPcd>
                 <cam_x>${cam_x}</cam_x>
                 <cam_y>${cam_y}</cam_y>

File: rotors_description/urdf/gcs.xacro (robot description, xacro)
@@ -22,5 +22,5 @@
   <xacro:property name="ppcom_config"     value="$(arg ppcom_config)" />
   <xacro:property name="ppcom_hz"         value="$(arg ppcom_hz)" />
-  <xacro:property name="interest_config"  value="$(arg interest_config)" />
+  <xacro:property name="interest_points"  value="$(arg interest_points)" />
   <xacro:property name="use_mesh_file"    value="true" />
   <xacro:property name="mesh_file"        value="package://rotors_description/meshes/gcs/gcs.dae" />
@@ -67,5 +67,5 @@
       ppcom_config="${ppcom_config}"
       ppcom_hz="${ppcom_hz}"
-      interest_config="${interest_config}"
+      interest_points="${interest_points}"
   >
     <inertia ixx="0.00001" ixy="0.0" ixz="0.0" iyy="0.00001" iyz="0.0" izz="0.00001" />
@@ -77,5 +77,5 @@
       mass="0.015"
       ppcom_config="${ppcom_config}"
-      interest_config="${interest_config}"
+      interest_points="${interest_points}"
       ppcom_topic="ppcom"
       ppcom_hz="${ppcom_hz}"
