Commit message: update drone model param

File: rotors_description/urdf/caric_photographer_base.xacro (robot description, xacro)
@@ -29,6 +29,6 @@
   <xacro:property name="rotor_offset_top" value="0.037" /> <!-- [m] -->
   <xacro:property name="radius_rotor" value="0.1" /> <!-- [m] -->
-  <xacro:property name="motor_constant" value="8.54858e-06" /> <!-- [kg m/s^2] -->
-  <xacro:property name="moment_constant" value="0.016" /> <!-- [m] -->
+  <xacro:property name="motor_constant" value="0.00002564574" /> <!-- [kg m/s^2] -->
+  <xacro:property name="moment_constant" value="0.048" /> <!-- [m] -->
   <xacro:property name="time_constant_up" value="0.0125" /> <!-- [s] -->
   <xacro:property name="time_constant_down" value="0.025" /> <!-- [s] -->
