Commit message: update model params

File: rotors_description/urdf/caric_explorer.xacro (robot description, xacro)
@@ -41,5 +41,5 @@
     rotating_period="8.0"
   >
-    <origin xyz="0.2 0 0.2" rpy="0 0 0" />
+    <origin xyz="0.0 0 0.2" rpy="0 0 0" />
     <inertia ixx="0.00001" ixy="0.0" ixz="0.0" iyy="0.00001" iyz="0.0" izz="0.00001" />
   </xacro:servo>

File: rotors_description/urdf/caric_explorer_base.xacro (robot description, xacro)
@@ -29,5 +29,5 @@
   <xacro:property name="rotor_offset_top" value="0.074" /> <!-- [m] -->
   <xacro:property name="radius_rotor" value="0.2" /> <!-- [m] -->
-  <xacro:property name="motor_constant" value="1.709716e-05" /> <!-- [kg m/s^2] -->
+  <xacro:property name="motor_constant" value="0.00002564574" /> <!-- [kg m/s^2] -->
   <xacro:property name="moment_constant" value="0.032" /> <!-- [m] -->
   <xacro:property name="time_constant_up" value="0.0125" /> <!-- [s] -->
