Commit message: update explorer parameter

File: rotors_description/urdf/caric_explorer_base.xacro (robot description, xacro)
@@ -33,5 +33,5 @@
   <xacro:property name="time_constant_up" value="0.0125" /> <!-- [s] -->
   <xacro:property name="time_constant_down" value="0.025" /> <!-- [s] -->
-  <xacro:property name="max_rot_velocity" value="1200" /> <!-- [rad/s] -->
+  <xacro:property name="max_rot_velocity" value="900" /> <!-- [rad/s] -->
   <xacro:property name="sin30" value="0.5" />
   <xacro:property name="cos30" value="0.866025403784" />
@@ -40,5 +40,5 @@
   <!-- Property Blocks -->
   <xacro:property name="body_inertia">
-    <inertia ixx="${2.5/1.5*0.0347563}" ixy="0.0" ixz="0.0" iyy="${2.5/1.5*0.0458929}" iyz="0.0" izz="${2.5/1.5*0.0977}" /> <!-- [kg m^2] [kg m^2] [kg m^2] [kg m^2] [kg m^2] [kg m^2] -->
+    <inertia ixx="${2.5/1.5*0.0458929}" ixy="0.0" ixz="0.0" iyy="${2.5/1.5*0.0458929}" iyz="0.0" izz="${2.5/1.5*0.0977}" /> <!-- [kg m^2] [kg m^2] [kg m^2] [kg m^2] [kg m^2] [kg m^2] -->
   </xacro:property>
   <!-- inertia of a single rotor, assuming it is a cuboid. Height=3mm, width=15mm -->
